File: kfly_hat.kicad_pcb (KiCad board)
At the start: 2 copper layers, 88 parts, among them J1 KFly_RC_Out, J10 KFly_RC_In, J11 swd-4, J12 Dronecode_GPS, J13 Dronecode_CAN, J14 Pixhawk_Switch, J2 KFly_RC_Out, J3 KFly_RC_Out, J4 KFly_RC_Out, J5 KFly_RC_Out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

Commit message: More PCB
Parts:
- J1, J10, J13, J5, J6, J7, R11, R12, R13, R14, R15, R16, R17, R18, R19, R3, R4, R5, R6, R7, R8, R9: moved to B.Cu
- MK1, MK2: footprint MountingHole:MountingHole_3.2mm_M3 -> MountingHole:MountingHole_3.2mm_M3_Pad_Via
- U9: footprint Package_DFN_QFN:DFN-8-1EP_3x3mm_P0.65mm_EP1.55x2.4mm -> dfn:DFN-8-1EP_3x3mm_P0.65mm_EP1.55x2.4mm
- moved C6 82.7 mm to (92.8, 59.8), turned to 90 degrees
- moved C11 82.0 mm to (90.9, 56.9), turned to 90 degrees
- moved J10 81.8 mm to (86.4, 106.9), turned to 270 degrees
- moved C7 79.4 mm to (97.3, 59.8), turned to 90 degrees
- moved C23 75.8 mm to (93.2, 63.4)
- moved C12 75.5 mm to (90.8, 59.4)
- moved C13 74.7 mm to (95.3, 59.4)
- moved C9 74.2 mm to (90.4, 62.6), turned to 180 degrees
- moved C16 74.1 mm to (90.1, 72.5), turned to 90 degrees
- moved U4 73.0 mm to (98.6, 96.7), turned to 90 degrees
- moved R4 72.9 mm to (97.8, 93.9), turned to 90 degrees
- moved U3 72.1 mm to (91.1, 87.4)
- moved R18 71.9 mm to (96.2, 93.9), turned to 90 degrees
- moved C10 70.9 mm to (93.1, 61.5)
- moved J3 70.4 mm to (86.4, 58.9), turned to 90 degrees
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Routing:
- net /HEAT: track 0.00 -> 28.2 mm
Other:
- board outline added: 35 x 56 mm
- copper layers 2 -> 4
- net class Default: trace_width 0.25 -> 0.2; via_dia 0.8 -> 0.6; via_drill 0.4 -> 0.3
- rule pad_to_mask_clearance: 0.2 -> 0.07

Commit message: More PCB
Parts:
- added R33: 10k, passive:R_0402_1005Metric_Rounded, F.Cu at (115.5, 108.5)
- added R34: 10k, passive:R_0402_1005Metric_Rounded, F.Cu at (115.5, 107.1)
- MK1, MK2: footprint MountingHole:MountingHole_3.2mm_M3_Pad_Via -> MountingHole:MountingHole_2.7mm_Pad_Via
- moved U2 81.4 mm to (77.4, 64.4)
- moved U8 72.4 mm to (71.4, 74.0), turned to 180 degrees
- moved D2 53.9 mm to (116.1, 116.4)
- moved D3 41.9 mm to (116.1, 114.4)
- moved R23 40.1 mm to (118.6, 114.4), turned to 180 degrees
- moved R22 39.7 mm to (118.6, 116.4), turned to 180 degrees
- moved D4 33.5 mm to (116.1, 112.4)
- moved X1 32.0 mm to (109.8, 70.2), turned to 270 degrees
- moved R32 24.1 mm to (118.6, 112.4)
- moved R26 17.5 mm to (108.1, 99.4), turned to 270 degrees
- moved U9 1.12 mm to (111.1, 99.4)

Commit message: More PCB
Parts:
- C19, C22, C5, C8, J11, R21, R26, U2, U5, U8, U9, X1: moved to B.Cu
- moved R10 79.7 mm to (80.5, 81.7)
- moved C19 76.4 mm to (91.6, 83.5), turned to 180 degrees
- moved C18 74.3 mm to (91.8, 90.8), turned to 270 degrees
- moved U5 73.9 mm to (97.0, 71.5), turned to 90 degrees
- moved R24 72.1 mm to (93.7, 57.7), turned to 270 degrees
- moved R21 71.8 mm to (95.5, 65.2), turned to 180 degrees
- moved C8 70.7 mm to (93.8, 67.1), turned to 270 degrees
- moved C5 70.5 mm to (98.7, 71.5), turned to 270 degrees
- moved C22 68.6 mm to (93.9, 86.4), turned to 270 degrees
- moved R25 67.0 mm to (95.0, 63.4), turned to 180 degrees
- moved C14 66.2 mm to (90.1, 69.5), turned to 90 degrees
- moved Q2 66.1 mm to (91.1, 87.7)
- moved R20 61.9 mm to (97.3, 61.9), turned to 270 degrees
- moved C1 61.5 mm to (102.3, 87.3), turned to 270 degrees
- moved R27 59.1 mm to (90.5, 90.4)
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Routing:
- net /HEAT: track 28.2 -> 0.00 mm
- net /COM_RX: track 0.00 -> 16.5 mm
- net /COM_TX: track 0.00 -> 13.8 mm
- net VAA: track 0.00 -> 4.27 mm
- net GND: vias 0 -> 20
Other:
- board size 35 x 56 mm -> 34.5 x 56 mm
